File: openPlc_Rpi.sch (KiCad schematic (older format))
At the start: 113 parts, among them J1 Raspberry_Pi_2_3, J10 Conn_01x04, J11 Conn_01x04, J12 Conn_01x04, J13 Conn_01x04, J14 Screw_Terminal_01x10, J3 Screw_Terminal_01x04, J4 Screw_Terminal_01x02, J5 Screw_Terminal_01x12, J7 Screw_Terminal_01x12, J8 Screw_Terminal_01x02, J9 Screw_Terminal_01x02, K1 G5LE-1, K2 G5LE-1, K3 G5LE-1, K4 G5LE-1, K5 G5LE-1, K6 G5LE-1, K7 G5LE-1, K8 G5LE-1, Q1 BSS123, Q2 2N7002, Q3 2N7002, U1 power_LM2576, U2 LTV-847, U3 LTV-847, U4 power_L7812_smd, U5 MAX481E, U6 ADS1018IDGS, U7 AMS1117-3.3, U8 ULN2803A

Commit message: [vishnu] created branch revision_0 and first commit to it.
Parts:
- removed R? (x2): R, symbol Device:R
Changed lines of the file:
@@
 	1    0    0    -1
 $EndComp
-$Comp
-L Device:R R?
-U 1 1 5E0E6830
-P 10950 10100
-F 0 "R?" H 11020 10146 50  0000 L CNN
-F 1 "R" H 11020 10055 50  0000 L CNN
-F 2 "" V 10880 10100 50  0001 C CNN
-F 3 "~" H 10950 10100 50  0001 C CNN
-	1    10950 10100
-	1    0    0    -1
-$EndComp
-$Comp
-L Device:R R?
-U 1 1 5E0F141A
-P 11550 10100
-F 0 "R?" H 11620 10146 50  0000 L CNN
-F 1 "R" H 11620 10055 50  0000 L CNN
-F 2 "" V 11480 10100 50  0001 C CNN
-F 3 "~" H 11550 10100 50  0001 C CNN
-	1    11550 10100
-	1    0    0    -1
-$EndComp
-Wire Wire Line
-	10950 9950 10950 9800
-Wire Wire Line
-	10950 9800 11550 9800
-Wire Wire Line
-	11550 9800 11550 9950
-Wire Wire Line
-	11550 10250 11550 10350
-Wire Wire Line
-	11550 10350 10950 10350
-Wire Wire Line
-	10950 10350 10950 10250
 $EndSCHEMATC

Commit message: fixed untracked files
Parts:
- added U9: 14528, symbol 4xxx:14528
Connections:
- wire segments 429 -> 438
- no-connect marks 5 -> 4
Changed lines of the file:
@@
 	1    0    0    -1
 $EndComp
-NoConn ~ 9550 11450
 $Comp
 L pspice:DIODE D19
@@
 	1    0    0    -1
 $EndComp
+$Comp
+L 4xxx:14528 U9
+U 1 1 5E168E86
+P 9350 11100
+F 0 "U9" H 9350 11567 50  0000 C CNN
+F 1 "14528" H 9350 11476 50  0000 C CNN
+F 2 "" H 9350 11100 50  0001 C CNN
+F 3 "https://www.onsemi.com/pub/Collateral/MC14528B-D.PDF" H 9350 11100 50  0001 C CNN
+	1    9350 11100
+	1    0    0    -1
+$EndComp
+Wire Wire Line
+	9850 11000 9950 11000
+Wire Wire Line
+	10200 11000 10200 11300
+Wire Wire Line
+	10200 11300 9850 11300
+Wire Wire Line
+	8850 11400 8850 11200
+Connection ~ 8850 11100
+Wire Wire Line
+	8850 11100 8850 10900
+Connection ~ 8850 11200
+Wire Wire Line
+	8850 11200 8850 11100
+Wire Wire Line
+	9350 11700 9950 11700
+Wire Wire Line
+	9950 11700 9950 11000
+Connection ~ 9950 11000
+Wire Wire Line
+	9950 11000 10200 11000
 $EndSCHEMATC
