File: openPlc_Rpi.sch (KiCad schematic (older format))
At the start: 112 parts, among them J1 Raspberry_Pi_2_3, J10 Conn_01x04, J11 Conn_01x04, J12 Conn_01x04, J13 Conn_01x04, J14 Screw_Terminal_01x10, J3 Screw_Terminal_01x04, J4 Screw_Terminal_01x02, J5 Screw_Terminal_01x12, J7 Screw_Terminal_01x12, J8 Screw_Terminal_01x02, J9 Screw_Terminal_01x02, K1 G5LE-1, K2 G5LE-1, K3 G5LE-1, K4 G5LE-1, K5 G5LE-1, K6 G5LE-1, K7 G5LE-1, K8 G5LE-1, Q1 BSS123, Q2 2N7002, Q3 2N7002, U1 power_LM2576, U2 LTV-847, U3 LTV-847, U4 power_L7812_smd, U5 MAX481E, U6 ADS1018IDGS, U7 AMS1117-3.3, U8 ULN2803A, U9 14528

Commit message: [vishnu] 	- removed the test circuit from the scematic
Parts:
- removed U9: 14528, symbol 4xxx:14528
Connections:
- wire segments 438 -> 429
Changed lines of the file:
@@
 	1    0    0    -1
 $EndComp
-$Comp
-L 4xxx:14528 U9
-U 1 1 5E168E86
-P 9350 11100
-F 0 "U9" H 9350 11567 50  0000 C CNN
-F 1 "14528" H 9350 11476 50  0000 C CNN
-F 2 "" H 9350 11100 50  0001 C CNN
-F 3 "https://www.onsemi.com/pub/Collateral/MC14528B-D.PDF" H 9350 11100 50  0001 C CNN
-	1    9350 11100
-	1    0    0    -1
-$EndComp
-Wire Wire Line
-	9850 11000 9950 11000
-Wire Wire Line
-	10200 11000 10200 11300
-Wire Wire Line
-	10200 11300 9850 11300
-Wire Wire Line
-	8850 11400 8850 11200
-Connection ~ 8850 11100
-Wire Wire Line
-	8850 11100 8850 10900
-Connection ~ 8850 11200
-Wire Wire Line
-	8850 11200 8850 11100
-Wire Wire Line
-	9350 11700 9950 11700
-Wire Wire Line
-	9950 11700 9950 11000
-Connection ~ 9950 11000
-Wire Wire Line
-	9950 11000 10200 11000
 Text Label 11100 6350 0    50   ~ 0
 TXD

Commit message: [vishnu] Corrected all footpronts to the present library version; PCB not updated.
Parts:
- C7: footprint Capacitors_SMD:C_1206_HandSoldering -> Capacitor_SMD:C_1206_3216Metric_Pad1.42x1.75mm_HandSolder
- D1, D10, D2, D3, D4, D7, D8, D9: footprint Diodes_SMD:D_1206 -> Diode_SMD:D_1206_3216Metric
- D11, D12, D13, D14, D15, D16, D17, D18: footprint LEDs:LED_0805_HandSoldering -> LED_SMD:LED_0805_2012Metric_Pad1.15x1.40mm_HandSolder
- D19: footprint Diodes_SMD:D_SMB_Handsoldering -> Diode_SMD:D_SMB_Handsoldering
- D5: footprint Diodes_SMD:D_SMA_Handsoldering -> Diode_SMD:D_SMA_Handsoldering
- D6: footprint Diodes_SMD:D_SMC_Handsoldering -> Diode_SMD:D_SMC_Handsoldering
- J1: footprint Socket_Strips:Socket_Strip_Straight_2x20_Pitch2.54mm -> Connector_PinSocket_2.54mm:PinSocket_2x20_P2.54mm_Vertical
- J10, J11, J12, J13: footprint Connectors_JST:JST_XH_B04B-XH-A_04x2.50mm_Straight -> Connector_JST:JST_XH_B4B-XH-A_1x04_P2.50mm_Vertical
- K1, K2, K3, K4, K5, K6, K7, K8: footprint Relays_THT:Relay_SPDT_OMRON-G5LE-1 -> Relay_THT:Relay_SPDT_Omron-G5LE-1
- L1: footprint Inductors_SMD:L_12x12mm_h6mm -> Inductor_SMD:L_12x12mm_H6mm
- Q1: footprint TO_SOT_Packages_SMD:SOT-23 -> Package_TO_SOT_SMD:SOT-23
- U1: footprint TO_SOT_Packages_SMD:TO-263-5_TabPin3 -> Package_TO_SOT_SMD:TO-263-5_TabPin3
- U2, U3: footprint Housings_DIP:DIP-16_W7.62mm_SMDSocket_SmallPads -> Package_DIP:DIP-16_W8.89mm_SMDSocket_LongPads
- U4: footprint TO_SOT_Packages_SMD:TO-263-2 -> Package_TO_SOT_SMD:TO-263-2
- U5: footprint Housings_SOIC:SOIC-8_3.9x4.9mm_Pitch1.27mm -> Package_SO:SOIC-8_3.9x4.9mm_P1.27mm
- U6: footprint Housings_SSOP:TSSOP-10_3x3mm_Pitch0.5mm -> Package_SO:TSSOP-10_3x3mm_P0.5mm
- U7: footprint TO_SOT_Packages_SMD:SOT-223-3_TabPin2 -> Package_TO_SOT_SMD:SOT-223-3_TabPin2
- U8: footprint Housings_SOIC:SOIC-18W_7.5x11.6mm_Pitch1.27mm -> Package_SO:SOIC-18W_7.5x11.6mm_P1.27mm

Commit message: [vishnu] created new standalone library for the project with all the necessary components and corresponding footprints.
Parts:
- J1: footprint Connector_PinSocket_2.54mm:PinSocket_2x20_P2.54mm_Vertical -> openPlc_Rpi:Raspberry_Pi_Zero_Socketed_THT_FaceUp_SingleMountingHoles_copy
Changed lines of the file:
@@
 F 0 "J1" H 12150 8900 50  0000 C CNN
 F 1 "Raspberry_Pi_2_3" H 12150 8800 50  0000 C CNN
-F 2 "Connector_PinSocket_2.54mm:PinSocket_2x20_P2.54mm_Vertical" H 12150 7250 50  0001 C CNN
+F 2 "openPlc_Rpi:Raspberry_Pi_Zero_Socketed_THT_FaceUp_SingleMountingHoles_copy" H 12150 7250 50  0001 C CNN
 F 3 "https://www.raspberrypi.org/documentation/hardware/raspberrypi/schematics/rpi_SCH_3bplus_1p0_reduced.pdf" H 12150 7250 50  0001 C CNN
 	1    12150 7250

Commit message: [vishnu] replaced Rpi symbol and footprint in schematic and pcb from the new library
Parts:
- removed J1: Raspberry_Pi_2_3, openPlc_Rpi:Raspberry_Pi_Zero_Socketed_THT_FaceUp_SingleMountingHoles_copy, symbol Connector:Raspberry_Pi_2_3
- added J1: Raspberry_Pi_2_3, fossee_openplc:Raspberry_Pi_Zero_FaceUp_SingleMountingHole, symbol fossee_openplc:Raspberry_Pi_2_3
Changed lines of the file:
@@
-	1    0    0    -1
-$EndComp
-$Comp
-L Connector:Raspberry_Pi_2_3 J1
-U 1 1 5BF3B5F0
-P 12150 7250
-F 0 "J1" H 12150 8900 50  0000 C CNN
-F 1 "Raspberry_Pi_2_3" H 12150 8800 50  0000 C CNN
-F 2 "openPlc_Rpi:Raspberry_Pi_Zero_Socketed_THT_FaceUp_SingleMountingHoles_copy" H 12150 7250 50  0001 C CNN
-F 3 "https://www.raspberrypi.org/documentation/hardware/raspberrypi/schematics/rpi_SCH_3bplus_1p0_reduced.pdf" H 12150 7250 50  0001 C CNN
-	1    12150 7250
 	1    0    0    -1
 $EndComp
@@
 Text GLabel 10900 7950 0    50   Input ~ 0
 DI_6
+$Comp
+L fossee_openplc:Raspberry_Pi_2_3 J1
+U 1 1 5E38381A
+P 12150 7250
+F 0 "J1" H 12150 8731 50  0000 C CNN
+F 1 "Raspberry_Pi_2_3" H 12150 8640 50  0000 C CNN
+F 2 "fossee_openplc:Raspberry_Pi_Zero_FaceUp_SingleMountingHole" H 12150 7250 50  0001 C CNN
+F 3 "https://www.raspberrypi.org/documentation/hardware/raspberrypi/schematics/rpi_SCH_3bplus_1p0_reduced.pdf" H 12150 7250 50  0001 C CNN
+	1    12150 7250
+	1    0    0    -1
+$EndComp
 $EndSCHEMATC

Commit message: [vishnu] replaced ADC circuit with new library components : scehmatic and PCB updated
Parts:
- removed C4: 100n, Capacitor_SMD:C_0805_2012Metric_Pad1.15x1.40mm_HandSolder, symbol Device:C
- removed J3: Screw_Terminal_01x04, TerminalBlock_Phoenix:TerminalBlock_Phoenix_MKDS-1,5-4-5.08_1x04_P5.08mm_Horizontal, symbol Connector:Screw_Terminal_01x04
- removed R10, R11, R12, R9: 10k, Resistor_SMD:R_0805_2012Metric_Pad1.15x1.40mm_HandSolder, symbol Device:R
- removed R13, R14, R15, R16: 5k, Resistor_SMD:R_0805_2012Metric_Pad1.15x1.40mm_HandSolder, symbol Device:R
- removed U6: ADS1018IDGS, Package_SO:TSSOP-10_3x3mm_P0.5mm, symbol Analog_ADC:ADS1018IDGS
- added C4: 100n, fossee_openplc:C_0805_2012Metric, symbol fossee_openplc:C_0805
- added J2: Screw_Terminal_01x04, fossee_openplc:TerminalBlock_Phoenix_MKDS-1,5-4-5.08_1x04_P5.08mm_Horizontal, symbol fossee_openplc:Screw_Terminal_01x04
- added R10, R11, R12, R9: 10k, fossee_openplc:R_0805_2012Metric_Pad1.15x1.40mm_HandSolder, symbol fossee_openplc:R_0805
- added R13, R14, R15, R16: 5k, fossee_openplc:R_0805_2012Metric_Pad1.15x1.40mm_HandSolder, symbol fossee_openplc:R_0805
- added U6: ADS1018IDGS, fossee_openplc:TSSOP-10_3x3mm_P0.5mm, symbol fossee_openplc:ADS1018IDGS

Commit message: [vishnu] Replaced all component in the POWER circuitry with local library components. Added tantalum, C_1206, AMS117 and ls812 parts to the library.
Parts:
- removed C2: 150uf, Capacitor_SMD:CP_Elec_8x10, symbol Device:CP
- removed C3: 1000uf, Capacitor_SMD:CP_Elec_10x10, symbol Device:CP
- removed D20: LED, LED_SMD:LED_0805_2012Metric_Pad1.15x1.40mm_HandSolder, symbol Device:LED
- removed D5: NTS245SF, Diode_SMD:D_SMA_Handsoldering, symbol Device:D_Zener
- removed D6: B340, Diode_SMD:D_SMC_Handsoldering, symbol dinkan:D_Schottky_power
- removed J4: Screw_Terminal_01x02, TerminalBlock_Phoenix:TerminalBlock_Phoenix_MKDS-1,5-2-5.08_1x02_P5.08mm_Horizontal, symbol Connector:Screw_Terminal_01x02
- removed L1: 680uh, Inductor_SMD:L_12x12mm_H6mm, symbol Device:L_Core_Ferrite
- removed R46: 220R, Resistor_SMD:R_0805_2012Metric_Pad1.15x1.40mm_HandSolder, symbol Device:R_US
- removed U1: power_LM2576, Package_TO_SOT_SMD:TO-263-5_TabPin3, symbol dinkan:power_LM2576
- added C2: 150uf, fossee_openplc:CP_Elec_8x10, symbol fossee_openplc:Capacitor_Polarized_8x10
- added C3: 1000uf, fossee_openplc:CP_Elec_10x10, symbol fossee_openplc:Capacitor_Polarized_10x10
- added D20: LED_ALT, fossee_openplc:LED_0805_2012Metric, symbol fossee_openplc:LED_ALT
- added D5: NTS245SF, fossee_openplc:D_SMA_Handsoldering, symbol fossee_openplc:D_Zener_SMA
- added D6: B340, fossee_openplc:D_SMC, symbol fossee_openplc:B340
- added J3: Screw_Terminal_01x02, fossee_openplc:TerminalBlock_Phoenix_MKDS-1,5-2-5.08_1x02_P5.08mm_Horizontal, symbol fossee_openplc:Screw_Terminal_01x02
- added L1: 680uh, fossee_openplc:L_12x12mm_H6mm, symbol fossee_openplc:L_Core_Ferrite_smd_12x12
- added R46: 220, fossee_openplc:R_0805_2012Metric_Pad1.15x1.40mm_HandSolder, symbol fossee_openplc:R_0805
- added U1: power_LM2576, fossee_openplc:TO-263-5_TabPin3, symbol fossee_openplc:power_LM2576
- C5, C6, C8: footprint Capacitor_SMD:C_0805_2012Metric_Pad1.15x1.40mm_HandSolder -> fossee_openplc:C_0805_2012Metric; symbol Device:C -> fossee_openplc:C_0805
- C7: footprint Capacitor_SMD:C_1206_3216Metric_Pad1.42x1.75mm_HandSolder -> fossee_openplc:C_1206_3216Metric_Pad1.42x1.75mm_HandSolder; symbol dinkan:Cap_tantalum_1206_3218 -> fossee_openplc:Cap_tantalum_1206_3218
- D19: footprint Diode_SMD:D_SMB_Handsoldering -> fossee_openplc:D_SMB; symbol pspice:DIODE -> fossee_openplc:D_SMB
- J10, J11, J13: footprint Connector_JST:JST_XH_B4B-XH-A_1x04_P2.50mm_Vertical -> fossee_openplc:JST_XH_B4B-XH-A_1x04_P2.50mm_Vertical; symbol Connector_Generic:Conn_01x04 -> fossee_openplc:JST_Conn_01x04
- U4: footprint Package_TO_SOT_SMD:TO-263-2 -> fossee_openplc:TO-263-2; symbol dinkan:power_L7812_smd -> fossee_openplc:power_L7812_smd
- U7: footprint Package_TO_SOT_SMD:SOT-223-3_TabPin2 -> fossee_openplc:SOT-223-3_TabPin2; symbol Regulator_Linear:AMS1117-3.3 -> fossee_openplc:AMS1117-3.3
Other:
- note removed: ".33uf"

Commit message: [vishnu] Replaced all components in the OUTPUT circuit with local library "fossee_openplc" parts. Deleted an outdated folder with SVG of the older version of the PCB.
Parts:
- C1: footprint Capacitor_SMD:C_0805_2012Metric_Pad1.15x1.40mm_HandSolder -> fossee_openplc:C_0805_2012Metric; symbol Device:C -> fossee_openplc:C_0805
- D1, D10, D2, D3, D4, D7, D8, D9: footprint Diode_SMD:D_1206_3216Metric -> fossee_openplc:D_1206_3216Metric; symbol Device:D_Zener -> fossee_openplc:D_Zener_1206
- D11, D12, D13, D14, D15, D16, D17, D18: footprint LED_SMD:LED_0805_2012Metric_Pad1.15x1.40mm_HandSolder -> fossee_openplc:LED_0805_2012Metric; symbol Device:LED -> fossee_openplc:LED_ALT
- J5, J7: footprint TerminalBlock_Phoenix:TerminalBlock_Phoenix_MKDS-1,5-12-5.08_1x12_P5.08mm_Horizontal -> fossee_openplc:TerminalBlock_Phoenix_MKDS-1,5-12-5.08_1x12_P5.08mm_Horizontal; symbol Connector:Screw_Terminal_01x12 -> fossee_openplc:Screw_Terminal_01x12
- K1, K2, K3, K4, K5, K6, K7, K8: footprint Relay_THT:Relay_SPDT_Omron-G5LE-1 -> fossee_openplc:Relay_SPDT_Omron-G5LE-1; symbol Relay:G5LE-1 -> fossee_openplc:relay_G5LE-1
- R33, R34, R35, R36, R37, R38, R39, R40: footprint Resistor_SMD:R_0805_2012Metric_Pad1.15x1.40mm_HandSolder -> fossee_openplc:R_0805_2012Metric_Pad1.15x1.40mm_HandSolder; symbol Device:R_US -> fossee_openplc:R_0805
- U8: footprint Package_SO:SOIC-18W_7.5x11.6mm_P1.27mm -> fossee_openplc:SOIC-18W_7.5x11.6mm_P1.27mm; symbol Transistor_Array:ULN2803A -> fossee_openplc:ULN2803A

Commit message: [vishnu] Replaced INPUT circuit with "fossee_openplc" components. Added *-bak and *.bash to gitignore.
Parts:
- J12: footprint Connector_JST:JST_XH_B4B-XH-A_1x04_P2.50mm_Vertical -> fossee_openplc:JST_XH_B4B-XH-A_1x04_P2.50mm_Vertical; symbol Connector_Generic:Conn_01x04 -> fossee_openplc:JST_Conn_01x04
- J14: footprint TerminalBlock_Phoenix:TerminalBlock_Phoenix_MKDS-1,5-10-5.08_1x10_P5.08mm_Horizontal -> fossee_openplc:TerminalBlock_Phoenix_MKDS-1,5-10-5.08_1x10_P5.08mm_Horizontal; symbol Connector:Screw_Terminal_01x10 -> fossee_openplc:Screw_Terminal_01x10
- R1, R17, R18, R19, R2, R20, R21, R22, R23, R24, R25, R26, R27, R28, R29, R3, R30, R31, R32, R4, R5, R6, R7, R8: footprint Resistor_SMD:R_0805_2012Metric_Pad1.15x1.40mm_HandSolder -> fossee_openplc:R_0805_2012Metric_Pad1.15x1.40mm_HandSolder; symbol Device:R -> fossee_openplc:R_0805
- U2, U3: footprint Package_DIP:DIP-16_W8.89mm_SMDSocket_LongPads -> fossee_openplc:DIP-16_W8.89mm_SMDSocket_LongPads; symbol Isolator:LTV-847 -> fossee_openplc:opt_isolator_PC847
