File: openPlc_Rpi.sch (KiCad schematic (older format))
At the start: 111 parts, among them J1 Raspberry_Pi_2_3, J10 Conn_01x04, J11 Conn_01x04, J12 Conn_01x04, J13 Conn_01x04, J14 Screw_Terminal_01x10, J2 Screw_Terminal_01x04, J3 Screw_Terminal_01x02, J5 Screw_Terminal_01x12, J7 Screw_Terminal_01x12, J8 Screw_Terminal_01x02, J9 Screw_Terminal_01x02, K1 G5LE-1, K2 G5LE-1, K3 G5LE-1, K4 G5LE-1, K5 G5LE-1, K6 G5LE-1, K7 G5LE-1, K8 G5LE-1, Q1 BSS123, Q2 2N7002, Q3 2N7002, U1 power_LM2576, U2 LTV-847, U3 LTV-847, U4 power_L7812_smd, U5 MAX481E, U6 ADS1018IDGS, U7 AMS1117-3.3, U8 ULN2803A

Commit message: [easwaran] rough draft of routing for new orientation completed with no unconnected ratnests.
Changed lines of the file:
@@
 	1    0    0    -1
 $EndComp
+Text GLabel 13850 6650 0    50   Input ~ 0
+SDA
 Text GLabel 13850 6750 0    50   Input ~ 0
-SDA
-Text GLabel 13850 6650 0    50   Input ~ 0
 SCL
 Text Notes 13650 6450 0    50   ~ 0

Commit message: [vishnu] 	- removed copper pours around relay input for better AC isolation. 	- did DRC and connected the missing labels of digital inputs.
Changed lines of the file:
@@
 Sheet 1 1
 Title "OpenPLC V2"
-Date ""
-Rev "0.1"
+Date "2020-05-27"
+Rev "0.1a"
 Comp "FOSSEE"
 Comment1 "by Vishnu  Easwaran E"
@@
 	5950 6700 6150 6700
 Connection ~ 5950 6700
-Text Label 6150 6700 0    50   ~ 0
-DI_0
-Text Label 6150 6150 0    50   ~ 0
-DI_1
-Text Label 6150 5600 0    50   ~ 0
-DI_2
-Text Label 6150 5050 0    50   ~ 0
-DI_3
 $Comp
 L fossee_openplc:D_Zener_1206 D7
@@
 Wire Wire Line
 	5950 9150 6150 9150
-Text Label 6150 9150 0    50   ~ 0
-DI_4
-Text Label 6150 8600 0    50   ~ 0
-DI_5
-Text Label 6150 8050 0    50   ~ 0
-DI_6
-Text Label 6150 7500 0    50   ~ 0
-DI_7
 $Comp
 L fossee_openplc:Screw_Terminal_01x12 J7
@@
 Text GLabel 10900 7850 0    50   Input ~ 0
 DI_0
-Text GLabel 13400 7150 2    50   Input ~ 0
-DI_3
-Text GLabel 13400 7050 2    50   Input ~ 0
-DI_4
 Text GLabel 10900 7450 0    50   Input ~ 0
 DI_5
@@
 Text GLabel 13400 8050 2    50   Input ~ 0
 DI_2
-Wire Wire Line
-	13400 8050 12950 8050
 Text GLabel 10900 7950 0    50   Input ~ 0
 DI_6
-$Comp
-L fossee_openplc:Raspberry_Pi_2_3 J1
-U 1 1 5E38381A
-P 12150 7250
-F 0 "J1" H 12150 8731 50  0000 C CNN
-F 1 "Raspberry_Pi_2_3" H 12150 8640 50  0000 C CNN
-F 2 "fossee_openplc:Raspberry_Pi_Zero_FaceUp_SingleMountingHole" H 12150 7250 50  0001 C CNN
-F 3 "https://www.raspberrypi.org/documentation/hardware/raspberrypi/schematics/rpi_SCH_3bplus_1p0_reduced.pdf" H 12150 7250 50  0001 C CNN
-	1    12150 7250
-	1    0    0    -1
-$EndComp
 Wire Wire Line
 	3500 12500 2900 12500
@@
 $EndComp
 $Comp
-L fossee_openplc:ADS1018IDGS U6
-U 1 1 5E5FDE16
-P 5400 13650
-F 0 "U6" H 5400 14331 50  0000 C CNN
-F 1 "ADS1018IDGS" H 5400 14240 50  0000 C CNN
-F 2 "fossee_openplc:TSSOP-10_3x3mm_P0.5mm" H 5350 13600 50  0001 C CNN
-F 3 "http://www.ti.com/lit/ds/symlink/ads1018.pdf" H 4500 14050 50  0001 C CNN
-	1    5400 13650
-	1    0    0    -1
-$EndComp
-$Comp
 L fossee_openplc:GND #PWR01
 U 1 1 5E63250D
@@
 	1    0    0    -1
 $EndComp
+$Comp
+L fossee_openplc:ADS1018IDGS U6
+U 1 1 5E5FDE16
+P 5400 13650
+F 0 "U6" H 5400 14331 50  0000 C CNN
+F 1 "ADS1018IDGS" H 5400 14240 50  0000 C CNN
+F 2 "fossee_openplc:TSSOP-10_3x3mm_P0.5mm" H 5350 13600 50  0001 C CNN
+F 3 "http://www.ti.com/lit/ds/symlink/ads1018.pdf" H 4500 14050 50  0001 C CNN
+	1    5400 13650
+	1    0    0    -1
+$EndComp
+$Comp
+L fossee_openplc:Raspberry_Pi_2_3 J1
+U 1 1 5E38381A
+P 12150 7250
+F 0 "J1" H 12150 8731 50  0000 C CNN
+F 1 "Raspberry_Pi_2_3" H 12150 8640 50  0000 C CNN
+F 2 "fossee_openplc:Raspberry_Pi_Zero_FaceUp_SingleMountingHole" H 12150 7250 50  0001 C CNN
+F 3 "https://www.raspberrypi.org/documentation/hardware/raspberrypi/schematics/rpi_SCH_3bplus_1p0_reduced.pdf" H 12150 7250 50  0001 C CNN
+	1    12150 7250
+	1    0    0    -1
+$EndComp
+Wire Wire Line
+	13400 8050 12950 8050
+Text GLabel 13400 7150 2    50   Input ~ 0
+DI_3
+Text GLabel 13400 7050 2    50   Input ~ 0
+DI_4
+Text GLabel 6150 7500 2    50   Input ~ 0
+DI_7
+Text GLabel 6150 6150 2    50   Input ~ 0
+DI_1
+Text GLabel 6150 8600 2    50   Input ~ 0
+DI_5
+Text GLabel 6150 6700 2    50   Input ~ 0
+DI_0
+Text GLabel 6150 8050 2    50   Input ~ 0
+DI_6
+Text GLabel 6150 5600 2    50   Input ~ 0
+DI_2
+Text GLabel 6150 5050 2    50   Input ~ 0
+DI_3
+Text GLabel 6150 9150 2    50   Input ~ 0
+DI_4
 $EndSCHEMATC

Commit message: [vishnu] added rpi 3d step models. moved opto and added the headers. updated the netlist.
Parts:
- added J15, J16, J4, J6: bergStrip_01x06_Male, fossee_openplc:bergStrip_male_1x06_P2.54mm_Vertical, symbol fossee_openplc:bergStrip_01x06_Male
Connections:
- net labels added: in_1, in_2, in_3, in_4, in_5, in_6, in_7, in_8
- wire segments 429 -> 433
- no-connect marks 4 -> 5
Changed lines of the file:
@@
 Wire Wire Line
 	19000 8550 19000 8750
-$Comp
-L fossee_openplc:Screw_Terminal_01x12 J5
-U 1 1 5C23AF1C
-P 21550 8850
-F 0 "J5" H 21630 8842 50  0000 L CNN
-F 1 "Screw_Terminal_01x12" V 21750 8400 50  0001 L CNN
-F 2 "fossee_openplc:TerminalBlock_Phoenix_MKDS-1,5-12-5.08_1x12_P5.08mm_Horizontal" H 21550 8850 50  0001 C CNN
-F 3 "~" H 21550 8850 50  0001 C CNN
-	1    21550 8850
-	1    0    0    -1
-$EndComp
-Text Label 21350 9250 2    50   Italic 0
+Text Label 20750 9250 2    50   Italic 0
 1
-Text Label 21350 9350 2    50   Italic 0
+Text Label 20750 9350 2    50   Italic 0
 2
-Text Label 21350 9450 2    50   Italic 0
+Text Label 20750 9450 2    50   Italic 0
 3
-Text Label 21350 8950 2    50   Italic 0
+Text Label 20750 8950 2    50   Italic 0
 4
-Text Label 21350 9050 2    50   Italic 0
+Text Label 20750 9050 2    50   Italic 0
 5
-Text Label 21350 9150 2    50   Italic 0
+Text Label 20750 9150 2    50   Italic 0
 6
-Text Label 21350 8650 2    50   Italic 0
+Text Label 20750 8650 2    50   Italic 0
 7
-Text Label 21350 8750 2    50   Italic 0
+Text Label 20750 8750 2    50   Italic 0
 8
-Text Label 21350 8850 2    50   Italic 0
+Text Label 20750 8850 2    50   Italic 0
 9
-Text Label 21350 8350 2    50   Italic 0
+Text Label 20750 8350 2    50   Italic 0
 10
-Text Label 21350 8450 2    50   Italic 0
+Text Label 20750 8450 2    50   Italic 0
 11
-Text Label 21350 8550 2    50   Italic 0
+Text Label 20750 8550 2    50   Italic 0
 12
 Text Label 19900 7350 0    50   Italic 0
@@
 L fossee_openplc:Screw_Terminal_01x12 J7
 U 1 1 5CBB002E
-P 21550 5600
-F 0 "J7" H 21630 5592 50  0000 L CNN
-F 1 "Screw_Terminal_01x12" V 21750 5150 50  0001 L CNN
-F 2 "fossee_openplc:TerminalBlock_Phoenix_MKDS-1,5-12-5.08_1x12_P5.08mm_Horizontal" H 21550 5600 50  0001 C CNN
-F 3 "~" H 21550 5600 50  0001 C CNN
-	1    21550 5600
-	1    0    0    -1
-$EndComp
-Text Label 21350 6000 2    50   ~ 0
+P 20900 5350
+F 0 "J7" H 20980 5342 50  0000 L CNN
+F 1 "Screw_Terminal_01x12" V 21100 4900 50  0001 L CNN
+F 2 "fossee_openplc:TerminalBlock_Phoenix_MKDS-1,5-12-5.08_1x12_P5.08mm_Horizontal" H 20900 5350 50  0001 C CNN
+F 3 "~" H 20900 5350 50  0001 C CNN
+	1    20900 5350
+	1    0    0    -1
+$EndComp
+Text Label 20700 5750 2    50   ~ 0
 13
-Text Label 21350 6100 2    50   ~ 0
+Text Label 20700 5850 2    50   ~ 0
 14
-Text Label 21350 6200 2    50   ~ 0
+Text Label 20700 5950 2    50   ~ 0
 15
-Text Label 21350 5700 2    50   ~ 0
+Text Label 20700 5450 2    50   ~ 0
 16
-Text Label 21350 5800 2    50   ~ 0
+Text Label 20700 5550 2    50   ~ 0
 17
-Text Label 21350 5900 2    50   ~ 0
+Text Label 20700 5650 2    50   ~ 0
 18
-Text Label 21350 5400 2    50   ~ 0
+Text Label 20700 5150 2    50   ~ 0
 19
-Text Label 21350 5500 2    50   ~ 0
+Text Label 20700 5250 2    50   ~ 0
 20
-Text Label 21350 5600 2    50   ~ 0
+Text Label 20700 5350 2    50   ~ 0
 21
-Text Label 21350 5100 2    50   ~ 0
+Text Label 20700 4850 2    50   ~ 0
 22
-Text Label 21350 5200 2    50   ~ 0
+Text Label 20700 4950 2    50   ~ 0
 23
-Text Label 21350 5300 2    50   ~ 0
+Text Label 20700 5050 2    50   ~ 0
 24
 Connection ~ 19500 3900
@@
 Text GLabel 6150 8050 2    50   Input ~ 0
 DI_6
-Text GLabel 6150 5600 2    50   Input ~ 0
-DI_2
 Text GLabel 6150 5050 2    50   Input ~ 0
 DI_3
 Text GLabel 6150 9150 2    50   Input ~ 0
 DI_4
+$Comp
+L fossee_openplc:bergStrip_01x06_Male J6
+U 1 1 5ED3F1FE
+P 6900 8350
+F 0 "J6" H 6872 8232 50  0000 R CNN
+F 1 "bergStrip_01x06_Male" H 6872 8323 50  0000 R CNN
+F 2 "fossee_openplc:bergStrip_male_1x06_P2.54mm_Vertical" H 6900 8350 50  0001 C CNN
+F 3 "~" H 6900 8350 50  0001 C CNN
+	1    6900 8350
+	-1   0    0    1
+$EndComp
+$Comp
+L fossee_openplc:Screw_Terminal_01x12 J5
+U 1 1 5C23AF1C
+P 20950 8850
+F 0 "J5" H 21030 8842 50  0000 L CNN
+F 1 "Screw_Terminal_01x12" V 21150 8400 50  0001 L CNN
+F 2 "fossee_openplc:TerminalBlock_Phoenix_MKDS-1,5-12-5.08_1x12_P5.08mm_Horizontal" H 20950 8850 50  0001 C CNN
+F 3 "~" H 20950 8850 50  0001 C CNN
+	1    20950 8850
+	1    0    0    -1
+$EndComp
+$Comp
+L fossee_openplc:bergStrip_01x06_Male J15
+U 1 1 5EE72B85
+P 17140 8970
+F 0 "J15" H 17112 8852 50  0000 R CNN
+F 1 "bergStrip_01x06_Male" H 17112 8943 50  0000 R CNN
+F 2 "fossee_openplc:bergStrip_male_1x06_P2.54mm_Vertical" H 17140 8970 50  0001 C CNN
+F 3 "~" H 17140 8970 50  0001 C CNN
+	1    17140 8970
+	-1   0    0    1
+$EndComp
+$Comp
+L fossee_openplc:bergStrip_01x06_Male J16
+U 1 1 5EE79333
+P 17180 5500
+F 0 "J16" H 17152 5382 50  0000 R CNN
+F 1 "bergStrip_01x06_Male" H 17152 5473 50  0000 R CNN
+F 2 "fossee_openplc:bergStrip_male_1x06_P2.54mm_Vertical" H 17180 5500 50  0001 C CNN
+F 3 "~" H 17180 5500 50  0001 C CNN
+	1    17180 5500
+	-1   0    0    1
+$EndComp
+Text GLabel 6150 5600 2    50   Input ~ 0
+DI_2
+Text GLabel 3150 7450 2    50   Input ~ 0
+in_1
+Text GLabel 3050 7350 2    50   Input ~ 0
+in_2
+Text GLabel 2900 7250 2    50   Input ~ 0
+in_3
+Text GLabel 2750 7150 2    50   Input ~ 0
+in_4
+Text GLabel 2750 6950 2    50   Input ~ 0
+in_5
+Text GLabel 2900 6850 2    50   Input ~ 0
+in_6
+Text GLabel 3050 6750 2    50   Input ~ 0
+in_7
+Text GLabel 3150 6650 2    50   Input ~ 0
+in_8
+Text GLabel 6700 5850 0    50   Input ~ 0
+in_8
+Text GLabel 6700 5950 0    50   Input ~ 0
+in_7
+Text GLabel 6700 6050 0    50   Input ~ 0
+in_6
+Text GLabel 6700 6150 0    50   Input ~ 0
+in_5
+Text GLabel 6700 8250 0    50   Input ~ 0
+in_4
+Text GLabel 6700 8350 0    50   Input ~ 0
+in_3
+Text GLabel 6700 8450 0    50   Input ~ 0
+in_2
+Text GLabel 6700 8550 0    50   Input ~ 0
+in_1
+$Comp
+L fossee_openplc:+5V #PWR0108
+U 1 1 5ED909B5
+P 6630 5650
+F 0 "#PWR0108" H 6630 5500 50  0001 C CNN
+F 1 "+5V" H 6645 5823 50  0000 C CNN
+F 2 "" H 6630 5650 50  0001 C CNN
+F 3 "" H 6630 5650 50  0001 C CNN
+	1    6630 5650
+	1    0    0    -1
+$EndComp
+$Comp
+L fossee_openplc:bergStrip_01x06_Male J4
+U 1 1 5ED3963E
+P 6900 5950
+F 0 "J4" H 6872 5832 50  0000 R CNN
+F 1 "bergStrip_01x06_Male" H 6872 5923 50  0000 R CNN
+F 2 "fossee_openplc:bergStrip_male_1x06_P2.54mm_Vertical" H 6900 5950 50  0001 C CNN
+F 3 "~" H 6900 5950 50  0001 C CNN
+	1    6900 5950
+	-1   0    0    1
+$EndComp
+Wire Wire Line
+	6700 5650 6630 5650
+$Comp
+L fossee_openplc:+5V #PWR0109
+U 1 1 5EE345BA
+P 6610 8050
+F 0 "#PWR0109" H 6610 7900 50  0001 C CNN
+F 1 "+5V" H 6625 8223 50  0000 C CNN
+F 2 "" H 6610 8050 50  0001 C CNN
+F 3 "" H 6610 8050 50  0001 C CNN
+	1    6610 8050
+	1    0    0    -1
+$EndComp
+Wire Wire Line
+	6610 8050 6700 8050
+$Comp
+L power:GND #PWR0110
+U 1 1 5EEABC0B
+P 6430 8150
+F 0 "#PWR0110" H 6430 7900 50  0001 C CNN
+F 1 "GND" H 6435 7977 50  0000 C CNN
+F 2 "" H 6430 8150 50  0001 C CNN
+F 3 "" H 6430 8150 50  0001 C CNN
+	1    6430 8150
+	1    0    0    -1
+$EndComp
+Wire Wire Line
+	6430 8150 6700 8150
+$Comp
+L power:GND #PWR0111
+U 1 1 5EEE0F26
+P 6410 5750
+F 0 "#PWR0111" H 6410 5500 50  0001 C CNN
+F 1 "GND" H 6415 5577 50  0000 C CNN
+F 2 "" H 6410 5750 50  0001 C CNN
+F 3 "" H 6410 5750 50  0001 C CNN
+	1    6410 5750
+	1    0    0    -1
+$EndComp
+Wire Wire Line
+	6410 5750 6700 5750
+NoConn ~ 6550 8010
 $EndSCHEMATC

Commit message: [vishnu] Added male headers at input and output. PCB updated. Labels updated.
Parts:
- removed J15, J16: bergStrip_01x06_Male, fossee_openplc:bergStrip_male_1x06_P2.54mm_Vertical, symbol fossee_openplc:bergStrip_01x06_Male
- added J15, J16: bergStrip_01x04_Male, fossee_openplc:bergStrip_1x04_P2.54mm_Vertical, symbol fossee_openplc:bergStrip_01x04_Male
Changed lines of the file:
@@
 	1    0    0    -1
-$EndComp
-$Comp
-L fossee_openplc:bergStrip_01x06_Male J15
-U 1 1 5EE72B85
-P 17140 8970
-F 0 "J15" H 17112 8852 50  0000 R CNN
-F 1 "bergStrip_01x06_Male" H 17112 8943 50  0000 R CNN
-F 2 "fossee_openplc:bergStrip_male_1x06_P2.54mm_Vertical" H 17140 8970 50  0001 C CNN
-F 3 "~" H 17140 8970 50  0001 C CNN
-	1    17140 8970
-	-1   0    0    1
-$EndComp
-$Comp
-L fossee_openplc:bergStrip_01x06_Male J16
-U 1 1 5EE79333
-P 17180 5500
-F 0 "J16" H 17152 5382 50  0000 R CNN
-F 1 "bergStrip_01x06_Male" H 17152 5473 50  0000 R CNN
-F 2 "fossee_openplc:bergStrip_male_1x06_P2.54mm_Vertical" H 17180 5500 50  0001 C CNN
-F 3 "~" H 17180 5500 50  0001 C CNN
-	1    17180 5500
-	-1   0    0    1
 $EndComp
 Text GLabel 6150 5600 2    50   Input ~ 0
@@
 	6410 5750 6700 5750
 NoConn ~ 6550 8010
+$Comp
+L fossee_openplc:bergStrip_01x04_Male J16
+U 1 1 5EDE97BC
+P 17310 8900
+F 0 "J16" H 17282 8782 50  0000 R CNN
+F 1 "bergStrip_01x04_Male" H 17880 9110 50  0000 R CNN
+F 2 "fossee_openplc:bergStrip_1x04_P2.54mm_Vertical" H 17310 8900 50  0001 C CNN
+F 3 "~" H 17310 8900 50  0001 C CNN
+	1    17310 8900
+	-1   0    0    1
+$EndComp
+$Comp
+L fossee_openplc:bergStrip_01x04_Male J15
+U 1 1 5EDF22C0
+P 17300 5500
+F 0 "J15" H 17272 5382 50  0000 R CNN
+F 1 "bergStrip_01x04_Male" H 17860 5700 50  0000 R CNN
+F 2 "fossee_openplc:bergStrip_1x04_P2.54mm_Vertical" H 17300 5500 50  0001 C CNN
+F 3 "~" H 17300 5500 50  0001 C CNN
+	1    17300 5500
+	-1   0    0    1
+$EndComp
+Text GLabel 17110 9000 0    39   Input ~ 0
+DO_0
+Text GLabel 17110 8900 0    39   Input ~ 0
+DO_1
+Text GLabel 17110 8800 0    39   Input ~ 0
+DO_2
+Text GLabel 17110 8700 0    39   Input ~ 0
+DO_3
+Text GLabel 17100 5600 0    39   Input ~ 0
+DO_4
+Text GLabel 17100 5400 0    39   Input ~ 0
+DO_6
+Text GLabel 17100 5300 0    39   Input ~ 0
+DO_7
+Text GLabel 17100 5500 0    39   Input ~ 0
+DO_5
 $EndSCHEMATC
